File: trackball.kicad_sch (KiCad schematic)
At the start: 202 parts, among them J1 Conn_01x02, J2 ZX-PM2.0-2-4PY, Q1 XR2302, Q2 XR2302, Q4 XR2302, SW1 HX TC-5608-Y, SW2 HX TC-5608-Y, SW3 HX TC-5608-Y, SW4 HX TC-5608-Y, SW5 HX TC-5608-Y, SW6 HX TC-5608-Y, SW7 HX TC-5608-Y, SW8 HX TC-5608-Y, SW9 TS-1010-C-A, U1 USB-TYPE-C-017, U10 WS2812B, U11 WS2812B, U12 WS2812B, U13 WS2812B, U14 WS2812B, U15 WS2812B, U16 WS2812B, U17 WS2812B, U18 WS2812B, U19 WS2812B, U2 SY80004DQD, U20 WS2812B, U21 WS2812B, U3 SY80004DQD, U4 PMW3610, U5 PMW3610, U6 WS2812B, U7 WS2812B, U8 WS2812B, U9 WS2812B, X1 XL7EL89CKI-111YLC-32M

Commit message: feat: rev.04 WIP
Parts:
- removed C64, C72: CGA0201X5R105M6R3ET, easyeda2kicad:C0201, symbol easyeda2kicad:CGA0201X5R105M6R3ET
- removed LED1, LED11, LED12, LED13, LED3, LED4, LED7, LED9: SZYY0402W, easyeda2kicad:LED0402-RD_WHITE, symbol easyeda2kicad:SZYY0402W
- removed Q4: XR2302, easyeda2kicad:SOT-23-3_L2.9-W1.3-P0.95-LS2.4-BR, symbol easyeda2kicad:XR2302
- removed R45, R46: RC-01W103JT, easyeda2kicad:R0201, symbol easyeda2kicad:RC-01W103JT
- removed R49, R53, R55, R60, R62, R64, R66, R68: RT0402BRE0750RL, easyeda2kicad:R0402, symbol easyeda2kicad:RT0402BRE0750RL
- added C35, C43: GRM155R60J226ME11D, easyeda2kicad:C0402, symbol easyeda2kicad:GRM155R60J226ME11D
- added R18: RT0402BRE0750RL, easyeda2kicad:R0402, symbol easyeda2kicad:RT0402BRE0750RL
Connections:
- net 3V3: now also C35.1, C43.1
- net D_RE1_GND: now also FPC6.4, FPC6.6
- net D_RE2_GND: now also FPC8.4, FPC8.6
- net GND: now also FPC5.3, FPC5.5, FPC7.3, FPC7.5, C35.2, C43.2, R18.1
- net MCU_VIB_EN: now also R18.2
- net MCU_BCKLT_EN: no longer names the net of U_MCU1.AD16 (P0.20)
- no-connect marks 51 -> 44
Other:
- moved on the sheet: C59, C62, C65, LED10, LED5, LED8, Q1, R48, R52, R61, R63, U10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
