File: trackball.kicad_sch (KiCad schematic)
At the start: 184 parts, among them J1 Conn_01x02, J2 ZX-PM2.0-2-4PY, Q1 XR2302, Q2 XR2302, SW1 HX TC-5608-Y, SW2 HX TC-5608-Y, SW3 HX TC-5608-Y, SW4 HX TC-5608-Y, SW5 HX TC-5608-Y, SW6 HX TC-5608-Y, SW7 HX TC-5608-Y, SW8 HX TC-5608-Y, SW9 TS-1010-C-A, U1 USB-TYPE-C-017, U10 WS2812B, U11 WS2812B, U12 WS2812B, U13 WS2812B, U14 WS2812B, U15 WS2812B, U16 WS2812B, U17 WS2812B, U18 WS2812B, U19 WS2812B, U2 SY80004DQD, U20 WS2812B, U21 WS2812B, U3 SY80004DQD, U4 PMW3610, U5 PMW3610, U6 WS2812B, U7 WS2812B, U8 WS2812B, U9 WS2812B, X1 XL7EL89CKI-111YLC-32M

Commit message: feat: rev.04 hardware
Parts:
- removed C61: 0201B103K160NT, easyeda2kicad:C0201, symbol easyeda2kicad:0201B103K160NT
- removed R23, R5: 0201WMF1603TEE, easyeda2kicad:R0201, symbol easyeda2kicad:0201WMF1603TEE
- removed R6, R7, R8: RC-01W103JT, easyeda2kicad:R0201, symbol easyeda2kicad:RC-01W103JT
- added C44: 0201B821K500NT, easyeda2kicad:C0201, symbol easyeda2kicad:0201B821K500NT
- added R24: RC-01W103JT, easyeda2kicad:R0201, symbol easyeda2kicad:RC-01W103JT
- added R45, R46, R5: 715k, easyeda2kicad:R0201, symbol easyeda2kicad:RC-01W7153FT
- R3, R50, R51: value RC-01W103JT -> ~; LCSC Part C320848 -> C18164332
- renumbered FPC6 to ENC.ANY.1, FPC8 to ENC.ANY.2, FPC5 to ENC.L1, FPC7 to ENC.R1, FPC2 to SENS.ANY.1, FPC4 to SENS.ANY.2, FPC1 to SENS.L1, FPC3 to SENS.R1
Connections:
- net 1V8: now also R25.2, R28.2, R41.2, R42.2, R5.2; no longer R10.2
- net 3V3: now also R46.2; no longer R3.2
- net ADC_BAT: now also R3.1, C44.1; no longer R51.1
- net BAT_VCC: now also R3.2; no longer R51.2
- net D_RE1_1V8: no longer R25.2, R42.2
- net D_RE1_A: no longer R42.1
- net D_RE1_B: no longer R25.1
- net D_RE2_1V8: no longer R28.2, R41.2
- net D_RE2_A: no longer R41.1
- net D_RE2_B: no longer R28.1
- net GND: now also R10.1, R51.1, C44.2, R24.1
- net GNDS: now also R51.2
- net RE1_A: now also R42.1
- net RE1_B: now also R25.1
- net RE2_A: now also R28.1
- net RE2_B: now also R41.1
- net at C6.1, U2.3 (FB): now also R24.2, R5.1; no longer R10.1
- net at C71.1, U3.3 (FB): now also R10.2, R45.1
- new net: R45.2, R46.1
Other:
- note added: "1.85V"
- note removed: "1.8V"
- note removed: "actually 1.875V to ensure no need in voltage level converter and for red LEDs"
- note removed: "actually 3.15V: should be still in CC range for RGB LEDs this whole power rail might be not populated if backlight and RGB aren't required"
- moved on the sheet: C16, C31, R21, R22, R25, R35, R36, R42, R51, U_RE1, U_RE2

Commit message: feat: 1k dongle, rev5 hw (wip)
Parts:
- removed C16, C30, C31: 0201B103K160NT, easyeda2kicad:C0201, symbol easyeda2kicad:0201B103K160NT
- removed J2: ZX-PM2.0-2-4PY, easyeda2kicad:HDR-TH_8P-P2.00-V-F-R2-C4-S2.00, symbol easyeda2kicad:ZX-PM2.0-2-4PY
- removed R12, R13, R14, R21, R35: RC-01W103JT, easyeda2kicad:R0201, symbol easyeda2kicad:RC-01W103JT
- removed R18: RT0402BRE0750RL, easyeda2kicad:R0402, symbol easyeda2kicad:RT0402BRE0750RL
- removed R22, R36: 0201WMF1603TEE, easyeda2kicad:R0201, symbol easyeda2kicad:0201WMF1603TEE
- removed U_RE1, U_RE2: GT-EVA01AA-L1, easyeda2kicad:RES-ADJ-SMD_GT-EVA01AA-L1, symbol easyeda2kicad:GT-EVA01AA-L1
- added C30: 0201B821K500NT, easyeda2kicad:C0201, symbol easyeda2kicad:0201B821K500NT
- added C61, C64: GRM155R60J226ME11D, easyeda2kicad:C0402, symbol easyeda2kicad:GRM155R60J226ME11D
- added ENC1, ENC2: EC05E1220401, easyeda2kicad:SW-SMD_EC05E1220401, symbol easyeda2kicad:EC05E1220401
- added J2: AFH34-S08FIA-1H, easyeda2kicad:FPC-SMD_8P-P0.50_JS_AFH34-S08FIA-1H, symbol easyeda2kicad:AFH34-S08FIA-1H
- added Q3: AO3415A_C5350990, easyeda2kicad:SOT-23-3_L2.9-W1.6-P1.90-LS2.8-BR, symbol easyeda2kicad:AO3415A_C5350990
- added Q4: XR2302, easyeda2kicad:SOT-23-3_L2.9-W1.3-P0.95-LS2.4-BR, symbol easyeda2kicad:XR2302
- added R12, R13, R14, R21, R22: RC0201JR-075K1L, easyeda2kicad:R0201, symbol easyeda2kicad:RC0201JR-075K1L
- added R18, R49, R6, R7, R8: RC-01W103JT, easyeda2kicad:R0201, symbol easyeda2kicad:RC-01W103JT
- added R23: 0201WMF1603TEE, easyeda2kicad:R0201, symbol easyeda2kicad:0201WMF1603TEE
- added U22: TPS2116DRLR, easyeda2kicad:SOT-583-8_L2.1-W1.6-P0.50-LS1.6-BL, symbol easyeda2kicad:TPS2116DRLR
Connections:
- net D_RE1_SW is gone; now on net D_RE1_GND: ENC.ANY.1.2
- net D_RE2_SW is gone; now on net D_RE2_GND: ENC.ANY.2.2
- net 1V8: now also J2.3, J2.7, R12.2, R13.1, R14.1
- net BAT_VCC: now also C61.1, Q3.2 (S), R7.2, U22.6 (VIN2); no longer C10.1, C7.1, R4.1, U_CHG1.7 (BATSENSN)
- net CHG_IRQ: now also R14.2
- net CHG_SCL: now also R13.2
- net CHG_SDA: now also R12.1
- net D_RE1_A: now also ENC1.A
- net D_RE1_B: now also ENC1.B
- net D_RE1_GND: now also ENC1.4, ENC1.5, ENC1.C
- net D_RE2_A: now also ENC2.A
- net D_RE2_B: now also ENC2.B
- net D_RE2_GND: now also ENC2.4, ENC2.5, ENC2.C
- net GND: now also ENC.L1.7, ENC.R1.7, SW9.3, SW9.4, C30.2, C61.2, C64.2, J2.1, J2.5, J2.6, Q4.2 (S), R21.2, R22.2, R49.1, R6.1, R8.1, U22.1 (GND)
- net MCU_RESET: now also J2.8
- net MCU_SWDCLK: now also J2.2
- net MCU_SWDIO: now also J2.4
- net MCU_VIB_EN: now also R6.2
- net MCU_WAKEUP: now also C30.1
- net SW1: no longer D2.2
- net SW2: no longer D2.1
- net SW3: no longer D3.2
- net SW4: no longer D3.1
- net SW5: no longer D4.2
- net SW6: no longer D4.1
- net SW7: no longer D5.2
- net SW8: no longer D5.1
- net USB_VBUS: now also Q4.1 (G), R18.2, R8.2, U22.3 (VIN1), U22.5 (MODE)
- net VSYS: no longer C15.1, C18.1, C3.1, C5.1, R15.2, R54.2, R65.2, U2.6 (IN), U3.6 (IN)
- net SW7_WK: now reaches R17.1, R40.1, SW7.1
- net SW7_WK: now also D5.2
- net SW4_WK: now reaches R29.1, R31.1, SW4.1
- net SW4_WK: now also D3.1
- net SW5_WK: now reaches R26.1, R33.1, SW5.1
- net SW5_WK: now also D4.2
- net SW6_WK: now reaches R27.1, R34.1, SW6.1
- net SW6_WK: now also D4.1
- net SW1_WK: now reaches R19.1, R37.1, SW1.1
- net SW1_WK: now also D2.2
- net SW3_WK: now reaches R30.1, R32.1, SW3.1
- net SW3_WK: now also D3.2
- net SW8_WK: now reaches R16.1, R39.1, SW8.1
- net SW8_WK: now also D5.1
- net SW2_WK: now reaches R20.1, R38.1, SW2.1
- net SW2_WK: now also D2.1
- net RE1_SW renamed ARB2
- net ARB2: no longer ENC.L1.7
- net RE2_SW renamed ARB1
- net ARB1: no longer ENC.R1.7
- net USB_CC1: no longer names the net of U1.A5 (CC1)
- net USB_CC1: now also R21.1; no longer U_CHG1.26 (CC1)
- net USB_CC2: no longer names the net of U1.B5 (CC2)
- net USB_CC2: now also R22.1; no longer U_CHG1.27 (CC2)
- new net: R23.1, R49.2
- new net: R18.1, R23.2, U22.4 (PR1)
- new net: C10.1, C7.1, Q3.3 (D), R4.1, U_CHG1.7 (BATSENSN)
- new net: Q3.1 (G), Q4.3 (D), R7.1
- new net VLOAD: C15.1, C18.1, C3.1, C5.1, C64.1, R15.2, R54.2, R65.2, U2.6 (IN), U22.2 (VOUT), U22.7 (VOUT), U3.6 (IN)
- no-connect marks 44 -> 43
Other:
- note added: "PD"
- moved on the sheet: AE1, BAT1, C10, C11, C12, C13, C14, C15, C17, C18, C19, C2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

Commit message: feat: rev7 hardware
Parts:
- removed C3: CGA0201X5R105M6R3ET, easyeda2kicad:C0201, symbol easyeda2kicad:CGA0201X5R105M6R3ET
- added C16, C3: CL31A107MQHNNNE, easyeda2kicad:C1206, symbol easyeda2kicad:CL31A107MQHNNNE
Connections:
- net 1V8: now also C16.1; no longer J2.7
- net ARB1: now also J2.5
- net ARB2: now also J2.6
- net GND: now also C16.2, C3.2; no longer J2.5, J2.6
- net USB_VBUS: no longer C1.1, R18.2, U22.3 (VIN1), U22.5 (MODE), U_MUX1.9 (VCC)
- net VLOAD: now also C3.1
- net VSYS: now also C1.1, R18.2, U22.3 (VIN1), U22.5 (MODE), U_MUX1.9 (VCC)
- net ARB3: now reaches U_MCU1.AD16 (P0.20)
- net ARB3: now also J2.7
- no-connect marks 43 -> 42
Other:
- note added: "https://efog.tech/storage/caps.jpeg"
- moved on the sheet: BAT1, C35, C43, C44, C59, C62, C65, C66, J1, J2, Q1, Q2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

Commit message: feat: rev7 hardware (final)
Parts:
- removed R18, R49: RC-01W103JT, easyeda2kicad:R0201, symbol easyeda2kicad:RC-01W103JT
- removed R23: 0201WMF1603TEE, easyeda2kicad:R0201, symbol easyeda2kicad:0201WMF1603TEE
- added R18: 715k, easyeda2kicad:R0201, symbol easyeda2kicad:RC-01W7153FT
- added R23: RC-01W103JT, easyeda2kicad:R0201, symbol easyeda2kicad:RC-01W103JT
- added R35: 0201WMF1603TEE, easyeda2kicad:R0201, symbol easyeda2kicad:0201WMF1603TEE
Connections:
- net GND: now also R23.2
- net VSYS: now also R18.1
- net at U22.4 (PR1): now also R23.1, R35.2
- new net: R18.2, R35.1
