File: trackball.kicad_sch (KiCad schematic)
At the start: 190 parts, among them J1 Conn_01x02, J2 AFH34-S08FIA-1H, Q1 XR2302, Q2 XR2302, Q3 AO3415A_C5350990, Q4 XR2302, SW1 HX TC-5608-Y, SW2 HX TC-5608-Y, SW3 HX TC-5608-Y, SW4 HX TC-5608-Y, SW5 HX TC-5608-Y, SW6 HX TC-5608-Y, SW7 HX TC-5608-Y, SW8 HX TC-5608-Y, SW9 TS-1010-C-A, U1 USB-TYPE-C-017, U10 WS2812B, U11 WS2812B, U12 WS2812B, U13 WS2812B, U14 WS2812B, U15 WS2812B, U16 WS2812B, U17 WS2812B, U18 WS2812B, U19 WS2812B, U2 SY80004DQD, U20 WS2812B, U21 WS2812B, U22 TPS2116DRLR, U3 SY80004DQD, U4 PMW3610, U5 PMW3610, U6 WS2812B, U7 WS2812B, U8 WS2812B, U9 WS2812B, X1 XL7EL89CKI-111YLC-32M

Commit message: feat: rev10 hardware
Parts:
- removed C10, C13, C61, C64: GRM155R60J226ME11D, easyeda2kicad:C0402, symbol easyeda2kicad:GRM155R60J226ME11D
- removed C11, C8: CL05A106MP5NUNC_C315248, easyeda2kicad:C0402, symbol easyeda2kicad:CL05A106MP5NUNC_C315248
- removed C12: 0201B103K160NT, easyeda2kicad:C0201, symbol easyeda2kicad:0201B103K160NT
- removed C3: CL31A107MQHNNNE, easyeda2kicad:C1206, symbol easyeda2kicad:CL31A107MQHNNNE
- removed C30: 0201B821K500NT, easyeda2kicad:C0201, symbol easyeda2kicad:0201B821K500NT
- removed C7, C9: CGA0201X5R105M6R3ET, easyeda2kicad:C0201, symbol easyeda2kicad:CGA0201X5R105M6R3ET
- removed D2, D3, D4, D5, D6, D7: BAS40-06T-7-F, easyeda2kicad:SC-75-3_L1.6-W0.8-P1.00-LS1.6-BR, symbol easyeda2kicad:BAS40-06T-7-F
- removed L2: FTC252012S1R0MBCD, easyeda2kicad:L1008, symbol easyeda2kicad:FTC252012S1R0MBCD
- removed Q3: AO3415A_C5350990, easyeda2kicad:SOT-23-3_L2.9-W1.6-P1.90-LS2.8-BR, symbol easyeda2kicad:AO3415A_C5350990
- removed Q4: XR2302, easyeda2kicad:SOT-23-3_L2.9-W1.3-P0.95-LS2.4-BR, symbol easyeda2kicad:XR2302
- removed R1, R11, R16, R17, R2, R25, R26, R27, R28, R31, R32, R35, R37, R38, R41, R42: 0201WMF1603TEE, easyeda2kicad:R0201, symbol easyeda2kicad:0201WMF1603TEE
- removed R12, R13, R14, R21, R22: RC0201JR-075K1L, easyeda2kicad:R0201, symbol easyeda2kicad:RC0201JR-075K1L
- removed R18: 715k, easyeda2kicad:R0201, symbol easyeda2kicad:RC-01W7153FT
- removed R3, R50, R51: ~, easyeda2kicad:R0201, symbol easyeda2kicad:RC-01W103JT
- removed R4: FRM121WFR010TM, easyeda2kicad:R1206, symbol easyeda2kicad:FRM121WFR010TM
- removed R56: RT0402BRE0750RL, easyeda2kicad:R0402, symbol easyeda2kicad:RT0402BRE0750RL
- removed R57, R7, R8: RC-01W103JT, easyeda2kicad:R0201, symbol easyeda2kicad:RC-01W103JT
- removed U22: TPS2116DRLR, easyeda2kicad:SOT-583-8_L2.1-W1.6-P0.50-LS1.6-BL, symbol easyeda2kicad:TPS2116DRLR
- removed U_CHG1: AXP2585, easyeda2kicad:QFN-32_L5.0-W5.0-P0.40-TL-EP2.9, symbol easyeda2kicad:AXP2585
- added C31, C67, C68: CL05A106MP5NUNC_C315248, easyeda2kicad:C0402, symbol easyeda2kicad:CL05A106MP5NUNC_C315248
- added C61, C64, C69: CGA0201X5R105M6R3ET, easyeda2kicad:C0201, symbol easyeda2kicad:CGA0201X5R105M6R3ET
- added C70: GRM155R60J226ME11D, easyeda2kicad:C0402, symbol easyeda2kicad:GRM155R60J226ME11D
- added L2, L6: FTC252012SR47MBCA, easyeda2kicad:IND-SMD_L2.5-W2.0, symbol easyeda2kicad:FTC252012SR47MBCA
- added R12, R18, R21, R22, R25, R26, R27, R28, R31, R32, R35, R37, R38, R41, R42, R60, R77, R78, R79, R80, R81: 0201WMF3403TEE, easyeda2kicad:R0201, symbol easyeda2kicad:RC-01W103JT
- added R36, R55, R58, R59, R62, R64, R66, R67, R68, R69, R70, R71, R72, R73, R74, R75, R76, R82: 0201WMF1002TEE, easyeda2kicad:R0201, symbol easyeda2kicad:RC-01W103JT
- added R49, R50, R51, R53, R7, R8: 715k, easyeda2kicad:R0201, symbol easyeda2kicad:RC-01W7153FT
- added U22: LP4034QVF, easyeda2kicad:DFN-10_L3.0-W3.0-P0.50-BL-EP2.5, symbol easyeda2kicad:LP4034QVF
- added U23: TPS2116DRLR, easyeda2kicad:SOT-583-8_L2.1-W1.6-P0.50-LS1.6-BL, symbol easyeda2kicad:TPS2116DRLR
- AE1: now left out of the parts list
- C16, SW1, SW2, SW3, SW4, SW5, SW6, SW7, SW8, U4, U5: now not fitted; now left out of the parts list
- C6, C71: value ~ -> (none)
- R10, R15, R23, R24, R43, R44, R6, R65: value RC-01W103JT -> 0201WMF3403TEE; LCSC Part C320848 -> C423573
- R19, R20, R29, R30, R33, R34, R39, R40, R47, R48, R52, R54: value RC-01W103JT -> 0201WMF1002TEE; LCSC Part C304504 -> C473048
Connections:
- net CHG_USBD_P is gone; now on net CHG_USBD: U_MUX1.2 (D2+)
- net GNDS is gone; now on net GND: U1.1, U1.2, U1.3, U1.4
- net VSYS is gone; now on net USB_VBUS: C1.1, U_MUX1.9 (VCC)
- net 1V8: now also R44.2, R18.1, R25.1, R26.2, R27.2, R28.1, R31.2, R32.2, R37.2, R38.2, R41.1, R59.1, R60.2; no longer R5.2
- net 3V3_EN: now also R12.2
- net ADC_BAT: now also R50.2, R51.1
- net BAT_TS: now also R55.2, R68.1, R70.2, R71.1, U22.4 (TS)
- net BAT_VCC: now also C68.2, L2.1, R53.2, U22.6 (BAT), U23.6 (VIN2)
- net CHG_ISACTIVE: now also U22.2 (STAT)
- net D_SS1_1V8: now also R7.2; no longer R43.2
- net D_SS1_RST: now also R7.1; no longer R43.1
- net D_SS2_1V8: now also R8.2; no longer R44.2
- net D_SS2_RST: now also R8.1; no longer R44.1
- net GND: now also R43.1, C31.1, C61.1, C67.1, C68.1, C69.1, C70.2, R12.1, R42.1, R49.1, R62.2, R64.2, R66.2, R67.2, R72.2, R77.2, R78.2, R79.2, R80.2, R81.1, U22.11 (GND), U22.5 (VSET), U23.1 (GND); no longer R23.2
- net RE1_A: now also R41.2
- net RE1_B: now also R18.2
- net RE2_A: now also R28.2
- net RE2_B: now also R25.2
- net SW1_WK: now also R26.1
- net SW2_WK: now also R27.1
- net SW3_WK: now also R32.1
- net SW4_WK: now also R31.1
- net SW5_WK: now also R37.1
- net SW6_WK: now also R38.1
- net SW7_WK: now also R60.1
- net SW8_WK: now also R44.1
- net USB_MUX_SEL: now also R43.2
- net USB_VBUS: now also C61.2, R21.2, U22.10 (VBUS), U23.3 (VIN1), U23.5 (MODE)
- net VLOAD: now also C70.1, U23.2 (VOUT), U23.7 (VOUT)
- net at U_MUX1.8 (~{OE}): now also R42.2
- net at U1.A5 (CC1): now also R62.1, R64.1
- net at U1.B5 (CC2): now also R66.1, R67.1
- net at R23.1: now also R35.2
- net CHG_IRQ renamed MCU_FASTCHG
- net MCU_FASTCHG: now also C69.2, R74.2, R75.2, R76.2
- net CHG_SCL: no longer names the net of U_MCU1.B17 (P0.23)
- net CHG_SDA: no longer names the net of U_MCU1.A20 (P0.25)
- net CHG_USBD_N renamed CHG_USBD
- new net: C31.2, R55.1, R70.1, U22.1 (REGN)
- new net: R58.1, R59.2
- new net: R5.2, R58.2
- new net: L2.2, L6.1
- new net: C64.1, L6.2, U22.7 (SW)
- new net: R81.2, R82.2
- new net: R21.1, R22.2
- new net: R49.2, R50.1
- new net: R68.2, R69.1, R71.2
- new net: R73.1, R77.1, R78.1, R79.1, R80.1, U22.3 (ISET)
- new net: R51.2, R53.1
- new net: R73.2, R74.1, R75.1, R76.1
- new net: R35.1, R36.1, U23.4 (PR1)
- new net: R36.2, R82.1
- new net: R69.2, R72.1
- new net: C64.2, U22.8 (BST)
- new net: R22.1, R23.2
- new net: C67.2, U22.9 (PMID)
- no-connect marks 42 -> 37
Other:
- note added: "Effects"
- note added: "OE (EN): active low SEL: low = D1, high = D2 ESD protection on all pins D2 = short for QC"
- note removed: "LEDs"
- note removed: "OE (EN): active low SEL: low = D1, high = D2 ESD protection on all pins"
- note removed: "PD"
- note removed: "concern: minimal LDO load? used only for I2C pullups (when LEDs are unpowered)"
- moved on the sheet: AE1, BAT1, C1, C14, C15, C17, C18, C19, C2, C20, C21, C22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
