File: trackball.kicad_pcb (KiCad board)
At the start: 6 copper layers, 65 x 85 mm, 247 parts, among them J2 AFH34-S08FIA-1H, Q1 XR2302, Q2 XR2302, Q3 AO3415A_C5350990, Q4 XR2302, SW1 HX TC-5608-Y, SW2 HX TC-5608-Y, SW3 HX TC-5608-Y, SW4 HX TC-5608-Y, SW5 HX TC-5608-Y, SW6 HX TC-5608-Y, SW7 HX TC-5608-Y, SW8 HX TC-5608-Y, SW9 TS-1010-C-A, U1 USB-TYPE-C-017, U10 WS2812B, U11 WS2812B, U12 WS2812B, U13 WS2812B, U14 WS2812B, U15 WS2812B, U16 WS2812B, U17 WS2812B, U18 WS2812B, U19 WS2812B, U2 SY80004DQD, U20 WS2812B, U21 WS2812B, U22 TPS2116DRLR, U3 SY80004DQD, U4 PMW3610, U5 PMW3610, U6 WS2812B, U7 WS2812B, U8 WS2812B, U9 WS2812B, X1 XL7EL89CKI-111YLC-32M

Commit message: chore: tidy
Parts:
- moved R32 1.29 mm to (38.7, 67.7)
- moved R5 0.05 mm to (36.7, 61.3)
Routing:
- net SW3_WK: track 19.8 -> 18.6 mm
- net 1V8: track 262.9 -> 262.0 mm, vias 33 -> 35
Other:
- board text added: "23/03/26"
- board text removed: "17/03/26"
