File: trackball.kicad_pcb (KiCad board)
At the start: 6 copper layers, 65 x 85 mm, 247 parts, among them J2 AFH34-S08FIA-1H, Q1 XR2302, Q2 XR2302, Q3 AO3415A_C5350990, Q4 XR2302, SW1 HX TC-5608-Y, SW2 HX TC-5608-Y, SW3 HX TC-5608-Y, SW4 HX TC-5608-Y, SW5 HX TC-5608-Y, SW6 HX TC-5608-Y, SW7 HX TC-5608-Y, SW8 HX TC-5608-Y, SW9 TS-1010-C-A, U1 USB-TYPE-C-017, U10 WS2812B, U11 WS2812B, U12 WS2812B, U13 WS2812B, U14 WS2812B, U15 WS2812B, U16 WS2812B, U17 WS2812B, U18 WS2812B, U19 WS2812B, U2 SY80004DQD, U20 WS2812B, U21 WS2812B, U22 TPS2116DRLR, U3 SY80004DQD, U4 PMW3610, U5 PMW3610, U6 WS2812B, U7 WS2812B, U8 WS2812B, U9 WS2812B, X1 XL7EL89CKI-111YLC-32M

Commit message: feat: rev10 hardware
Parts:
- removed C10, C13: GRM155R60J226ME11D, easyeda2kicad:C0402
- removed C11, C8: CL05A106MP5NUNC_C315248, easyeda2kicad:C0402
- removed C12: 0201B103K160NT, easyeda2kicad:C0201
- removed C3: CL31A107MQHNNNE, easyeda2kicad:C1206
- removed C7, C9: CGA0201X5R105M6R3ET, easyeda2kicad:C0201
- removed ENC2: EC05E1220401, easyeda2kicad:SW-SMD_EC05E1220401
- removed Q3: AO3415A_C5350990, easyeda2kicad:SOT-23-3_L2.9-W1.6-P1.90-LS2.8-BR
- removed Q4: XR2302, easyeda2kicad:SOT-23-3_L2.9-W1.3-P0.95-LS2.4-BR
- removed R1, R11, R16, R17, R2: 0201WMF1603TEE, easyeda2kicad:R0201
- removed R13, R14: RC0201JR-075K1L, easyeda2kicad:R0201
- removed R3: ~, easyeda2kicad:R0201
- removed R4: FRM121WFR010TM, easyeda2kicad:R1206
- removed U_CHG1: AXP2585, easyeda2kicad:QFN-32_L5.0-W5.0-P0.40-TL-EP2.9
- added C31: CL05A106MP5NUNC_C315248, easyeda2kicad:C0402, F.Cu at (42.0, 41.7)
- added C67: CL05A106MP5NUNC_C315248, easyeda2kicad:C0402, F.Cu at (46.2, 42.9)
- added C68: CL05A106MP5NUNC_C315248, easyeda2kicad:C0402, F.Cu at (39.4, 42.1)
- added C69: CGA0201X5R105M6R3ET, easyeda2kicad:C0201, F.Cu at (47.3, 55.1)
- added C70: GRM155R60J226ME11D, easyeda2kicad:C0402, F.Cu at (36.0, 57.1)
- added ENC1: EC05E1220401, easyeda2kicad:SW-SMD_EC05E1220401, F.Cu at (67.5, 78.2)
- added L6: FTC252012SR47MBCA, easyeda2kicad:IND-SMD_L2.5-W2.0, F.Cu at (43.0, 47.2)
- added R36: 0201WMF1002TEE, easyeda2kicad:R0201, F.Cu at (41.6, 55.1)
- added R49: 715k, easyeda2kicad:R0201, F.Cu at (75.9, 52.2)
- added R53: 715k, easyeda2kicad:R0201, F.Cu at (74.4, 54.4)
- added R55: 0201WMF1002TEE, easyeda2kicad:R0201, F.Cu at (41.4, 40.6)
- added R58: 0201WMF1002TEE, easyeda2kicad:R0201, F.Cu at (35.0, 61.1)
- added R59: 0201WMF1002TEE, easyeda2kicad:R0201, F.Cu at (36.4, 62.1)
- added R60: 0201WMF3403TEE, easyeda2kicad:R0201, F.Cu at (93.8, 82.1)
- added R62: 0201WMF1002TEE, easyeda2kicad:R0201, F.Cu at (70.1, 44.0)
- added R64: 0201WMF1002TEE, easyeda2kicad:R0201, F.Cu at (71.1, 45.0)
- added R66: 0201WMF1002TEE, easyeda2kicad:R0201, F.Cu at (57.6, 43.6)
- added R67: 0201WMF1002TEE, easyeda2kicad:R0201, F.Cu at (58.6, 42.8)
- added R68: 0201WMF1002TEE, easyeda2kicad:R0201, F.Cu at (40.0, 40.4)
- added R69: 0201WMF1002TEE, easyeda2kicad:R0201, F.Cu at (38.7, 38.6)
- added R70: 0201WMF1002TEE, easyeda2kicad:R0201, F.Cu at (41.4, 39.6)
- added R71: 0201WMF1002TEE, easyeda2kicad:R0201, F.Cu at (39.9, 39.4)
- added R72: 0201WMF1002TEE, easyeda2kicad:R0201, F.Cu at (38.7, 40.2)
- added R73: 0201WMF1002TEE, easyeda2kicad:R0201, F.Cu at (46.1, 52.5)
- added R74: 0201WMF1002TEE, easyeda2kicad:R0201, F.Cu at (46.1, 53.5)
- added R75: 0201WMF1002TEE, easyeda2kicad:R0201, F.Cu at (46.1, 54.5)
- added R76: 0201WMF1002TEE, easyeda2kicad:R0201, F.Cu at (46.1, 55.4)
- added R77: 0201WMF3403TEE, easyeda2kicad:R0201, F.Cu at (44.6, 55.4)
- added R78: 0201WMF3403TEE, easyeda2kicad:R0201, F.Cu at (44.7, 52.5)
- added R79: 0201WMF3403TEE, easyeda2kicad:R0201, F.Cu at (44.6, 53.5)
- added R80: 0201WMF3403TEE, easyeda2kicad:R0201, F.Cu at (44.6, 54.5)
- added R81: 0201WMF3403TEE, easyeda2kicad:R0201, F.Cu at (42.4, 53.9)
- added R82: 0201WMF1002TEE, easyeda2kicad:R0201, F.Cu at (41.4, 53.9)
- added U23: TPS2116DRLR, easyeda2kicad:SOT-583-8_L2.1-W1.6-P0.50-LS1.6-BL, F.Cu at (38.3, 56.0)
- C61, C64: value GRM155R60J226ME11D -> CGA0201X5R105M6R3ET; footprint easyeda2kicad:C0402 -> easyeda2kicad:C0201
- L2: value FTC252012S1R0MBCD -> FTC252012SR47MBCA; footprint easyeda2kicad:L1008 -> easyeda2kicad:IND-SMD_L2.5-W2.0
- R10, R15, R23, R24, R43, R44, R6, R65: value RC-01W103JT -> 0201WMF3403TEE
- R12, R21, R22: value RC0201JR-075K1L -> 0201WMF3403TEE
- R18: value 715k -> 0201WMF3403TEE
- R19, R20, R29, R30, R33, R34, R39, R40, R47, R48, R52, R54, R57: value RC-01W103JT -> 0201WMF1002TEE
- R25, R26, R27, R28, R31, R32, R35, R37, R38, R41, R42: value 0201WMF1603TEE -> 0201WMF3403TEE
- R50, R51: value ~ -> 715k
- R7, R8: value RC-01W103JT -> 715k
- U22: value TPS2116DRLR -> LP4034QVF; footprint easyeda2kicad:SOT-583-8_L2.1-W1.6-P0.50-LS1.6-BL -> easyeda2kicad:DFN-10_L3.0-W3.0-P0.50-BL-EP2.5
- moved R37 67.5 mm to (59.0, 120.4)
- moved R26 67.4 mm to (76.1, 55.3), turned to 0 degrees
- moved R12 65.5 mm to (35.5, 112.0)
- moved R8 64.2 mm to (80.5, 94.1)
- moved R38 61.4 mm to (64.9, 120.5), turned to 180 degrees
- moved R27 59.0 mm to (59.1, 59.3)
- moved R7 53.4 mm to (62.6, 94.1)
- moved R43 45.7 mm to (68.8, 48.8), turned to 0 degrees
- moved R51 38.1 mm to (75.9, 54.2), turned to 180 degrees
- moved R41 33.6 mm to (57.9, 54.0), turned to 0 degrees
- moved R21 30.0 mm to (41.6, 52.6), turned to 0 degrees
- moved R18 28.2 mm to (72.5, 58.7), turned to 180 degrees
- moved R22 21.2 mm to (40.2, 53.1), turned to 180 degrees
- moved R44 19.2 mm to (93.7, 80.1)
- moved R25 19.1 mm to (86.0, 61.6)
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- renumbered ENC.ANY.1 to ENC.ANY, ENC.ANY.2 to ENC.ANY, SENS.ANY.1 to SENS.ANY, SENS.ANY.2 to SENS.ANY
Connections:
- C1 pad 1: VSYS -> USB_VBUS
- C61 pad 1: BAT_VCC -> GND
- C61 pad 2: GND -> USB_VBUS
- C64 pad 1: VLOAD -> Net-(U22-SW)
- C64 pad 2: GND -> Net-(U22-BST)
- L2 pad 1: Net-(L2-Pad1) -> BAT_VCC
- L2 pad 2: VSYS -> Net-(L2-Pad2)
- R12 pad 1: CHG_SDA -> GND
- R12 pad 2: 1V8 -> 3V3_EN
- R18 pad 1: VSYS -> 1V8
- R18 pad 2: Net-(R18-Pad2) -> RE1_B
- R21 pad 1: Net-(U1-CC1) -> Net-(R21-Pad1)
- R21 pad 2: GND -> USB_VBUS
- R22 pad 1: Net-(U1-CC2) -> Net-(R22-Pad1)
- R22 pad 2: GND -> Net-(R21-Pad1)
- R23 pad 1: Net-(U22-PR1) -> Net-(R23-Pad1)
- R23 pad 2: GND -> Net-(R22-Pad1)
- R25 pad 1: RE1_B -> 1V8
- R25 pad 2: 1V8 -> RE2_B
- R26 pad 1: SW5_WK -> SW1_WK
- R27 pad 1: SW6_WK -> SW2_WK
- R28 pad 1: RE2_A -> 1V8
- R28 pad 2: 1V8 -> RE2_A
- R35 pad 1: Net-(R18-Pad2) -> Net-(U23-PR1)
- R35 pad 2: Net-(U22-PR1) -> Net-(R23-Pad1)
- R37 pad 1: SW1_WK -> SW5_WK
- R38 pad 1: SW2_WK -> SW6_WK
- R41 pad 1: RE2_B -> 1V8
- R41 pad 2: 1V8 -> RE1_A
- R42 pad 1: RE1_A -> GND
- R42 pad 2: 1V8 -> Net-(U_MUX1-~{OE})
- R43 pad 1: D_SS1_RST -> GND
- R43 pad 2: D_SS1_1V8 -> USB_MUX_SEL
- R44 pad 1: D_SS2_RST -> SW8_WK
- R44 pad 2: D_SS2_1V8 -> 1V8
- R5 pad 2: 1V8 -> Net-(R5-Pad2)
- R50 pad 1: GND -> Net-(R49-Pad2)
- R51 pad 1: GND -> ADC_BAT
- R51 pad 2: GNDS -> Net-(R51-Pad2)
- R7 pad 1: Net-(Q3-G) -> D_SS1_RST
- R7 pad 2: BAT_VCC -> D_SS1_1V8
- R8 pad 1: GND -> D_SS2_RST
- R8 pad 2: USB_VBUS -> D_SS2_1V8
- SENS.L pad 9: USB_VBUS -> (no net)
- U1 pad 1: GNDS -> GND
- U1 pad 2: GNDS -> GND
- U1 pad 3: GNDS -> GND
- U1 pad 4: GNDS -> GND
- U22 pad 1: GND -> Net-(U22-REGN)
- U22 pad 2: VLOAD -> CHG_ISACTIVE
- U22 pad 3: VSYS -> Net-(U22-ISET)
- U22 pad 4: Net-(U22-PR1) -> BAT_TS
- U22 pad 5: VSYS -> GND
- U22 pad 7: VLOAD -> Net-(U22-SW)
- U22 pad 8: unconnected-(U22-ST-Pad8) -> Net-(U22-BST)
- U_MCU1 pad A16: CHG_IRQ -> MCU_FASTCHG
- U_MCU1 pad A20: CHG_SDA -> unconnected-(U_MCU1-P0.25-PadA20)
- U_MCU1 pad B17: CHG_SCL -> unconnected-(U_MCU1-P0.23-PadB17)
- U_MUX1 pad 2: CHG_USBD_P -> CHG_USBD
- U_MUX1 pad 6: CHG_USBD_N -> CHG_USBD
- U_MUX1 pad 9: VSYS -> USB_VBUS
Routing:
- net GNDS: track 110.2 -> 0.00 mm, vias 6 -> 0
- net VSYS: track 62.1 -> 0.00 mm, vias 4 -> 0
- net CHG_IRQ: track 61.3 -> 0.00 mm, vias 2 -> 0
- net CHG_SCL: track 58.5 -> 0.00 mm, vias 2 -> 0
- net CHG_SDA: track 58.0 -> 0.00 mm, vias 2 -> 0
- net MCU_FASTCHG: track 0.00 -> 52.9 mm, vias 0 -> 2
- net 1V8: track 262.0 -> 217.1 mm, vias 35 -> 34
- net Net-(Q3-D): track 33.3 -> 0.00 mm, vias 4 -> 0
- net USB_VBUS: track 138.3 -> 163.8 mm
- net CHG_USBD_N: track 22.5 -> 0.00 mm, vias 2 -> 0
- net CHG_USBD_P: track 22.4 -> 0.00 mm, vias 2 -> 0
- net Net-(U22-ISET): track 0.00 -> 19.9 mm, vias 0 -> 2
- net Net-(U_CHG1-BATSENSP): track 19.8 -> 0.00 mm, vias 3 -> 0
- net VIB_GND: track 35.3 -> 15.7 mm
- net 3V3: track 145.6 -> 162.8 mm, vias 9 -> 14
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- added copper zone on In3.Cu, net GND
Other:
- board text added: "18 Aug 26"
- board text added: "Aug 2026"
- board text added: "rev. 10"
- board text removed: "23/03/26"
- board text removed: "Mar 2026"
- board text removed: "rev. 07"
