File: paw3395-upgrade/paw3395-bb.kicad_pcb (KiCad board)
At the start: 2 copper layers, 15 x 27.5 mm, 10 parts, among them J1 AFH34-S08FIA-1H, U1 PAW3395

Commit message: feat: rev7 hardware
Parts:
- moved C2 4.50 mm to (87.1, 156.8), turned to 0 degrees
- moved C3 1.55 mm to (88.9, 156.8)
- moved C5 0.61 mm to (84.5, 137.9)
- moved C6 0.61 mm to (85.9, 138.0)
- moved C4 0.30 mm to (88.2, 157.9)
Routing:
- net Net-(U1-VDDREG): track 7.39 -> 12.6 mm
- net 1V8: track 49.8 -> 54.7 mm, vias 3 -> 4
