File: dongle-1k/dongle.kicad_sch (KiCad schematic)
At the start: 23 parts, among them U1 NRF52833-QDAA-R7, U2 TSC4A 160GF-WZ 016, U3 XL-1010RGBC-WS2812B, X1 XL7EL89CKI-111YLC-32M

Commit message: feat: rev10 hardware
Parts:
- removed L1: LQP03TN6N2H02D, easyeda2kicad:L0201, symbol easyeda2kicad:LQP03TN6N2H02D
- removed L2: LQP03HQ4N0B02D, easyeda2kicad:L0201, symbol easyeda2kicad:LQP03HQ4N7H02D
- added L4: LQP03HQ2N2H02D, easyeda2kicad:L0201, symbol easyeda2kicad:LQP03HQ4N7H02D
- A1: value KH-3216-A35 -> (none); footprint easyeda2kicad:ANT-SMD-2_L3.2-W1.6-C504002 -> mifa:mifa-2.4ghz-fr4-2.0mm; LCSC Part C504002 -> (none); now left out of the parts list
Connections:
- net GND: now also A1.2
- net at C4.2, L3.2: now also L4.1
- net at A1.1: now also L4.2
- no-connect marks 15 -> 14
Other:
- moved on the sheet: A1
